File: LinePCB.kicad_sch (KiCad schematic)
At the start: 128 parts, among them J1 Conn_02x05_Odd_Even, J2 Conn_01x02, U1 MCP3008, U10 2200, U11 210, U12 Oprocoupler, U13 10k, U14 N channel, U15 D, U16 10K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

Commit message: Finished Placement
Parts:
- removed H4, H5, H6, H7, H8: MountingHole, MountingHole:MountingHole_3.2mm_M3_DIN965_Pad, symbol Mechanical:MountingHole
- U1, U2, U3: footprint MCP3008:SOIC16-N_MC_MCH-L -> footprints:SOIC16-N_MC_MCH-L
- U17: footprint SMDPads:Pads_1x02 -> SMDPads:Pads
